File: Multimeter/Multimeter.kicad_sch (KiCad schematic)
At the start: 22 parts, among them J1 POWER, J2 INPUT, J3 ADC, SW1 SW_DPDT_x2, SW2 SW_DPDT_x2, U1 NE555P

Commit message: Enabled protection diodes for SPICE and increased test spike voltage
Parts:
- D2, D3: Spice_Netlist_Enabled N -> Y
- V5: Spice_Model ac(1) pwl(0 0 25u 0 27u 400 31u -400 33u 0 50u 0 50.002u 50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 -> ac(1) pwl(0 0 25u 0 27u 1k 31u -1k 33u 0 50u 0 50.002u 50 1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
Changed lines of the file:
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@@
       (effects (font (size 1.27 1.27)) (justify left) hide)
     )
-    (property "Spice_Model" "ac(1) pwl(0 0 25u 0 27u 400 31u -400 33u 0 50u 0 50.002u 50 100u 50 100.002u -50 150u -50 150.002u 0 200u 0 250u 100 350u -100 400u 0)" (id 6) (at 218.44 123.19 0)
+    (property "Spice_Model" "ac(1) pwl(0 0 25u 0 27u 1k 31u -1k 33u 0 50u 0 50.002u 50 100u 50 100.002u -50 150u -50 150.002u 0 200u 0 250u 100 350u -100 400u 0)" (id 6) (at 218.44 123.19 0)
       (effects (font (size 1.27 1.27)) (justify left) hide)
     )
@@
       (effects (font (size 1.27 1.27)) hide)
     )
-    (property "Spice_Netlist_Enabled" "N" (id 6) (at 184.15 114.3 0)
+    (property "Spice_Netlist_Enabled" "Y" (id 6) (at 184.15 114.3 0)
       (effects (font (size 1.27 1.27)) hide)
     )
@@
       (effects (font (size 1.27 1.27)) hide)
     )
-    (property "Spice_Netlist_Enabled" "N" (id 6) (at 203.2 120.65 0)
-      (effects (font (size 1.27 1.27)) hide)
-    )
+    (property "Spice_Netlist_Enabled" "Y" (id 6) (at 203.2 120.65 0)
+      (effects (font (size 1.27 1.27)) hide)
+    )
